File: DNA/class_D/class_D_manual/analog_input.kicad_sch (KiCad schematic)
At the start: 12 parts, among them U1 OPA2192

Commit message: [DNA]: class D, more of schematics added.
Connections:
- net RNORM: now reaches C2.1, R3.2, U1.7
- net MID: now reaches R8.2
- net V_IN: now reaches R1.1
Other:
- moved on the sheet: R5, R6, R7, R8
Changed lines of the file:
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@@
   (junction (at 99.06 77.47) (diameter 0) (color 0 0 0 0)
   )
-  (junction (at 137.16 115.57) (diameter 0) (color 0 0 0 0)
-  )
   (junction (at 49.53 74.93) (diameter 0) (color 0 0 0 0)
   )
+  (junction (at 137.16 118.11) (diameter 0) (color 0 0 0 0)
+  )
   (junction (at 185.42 80.01) (diameter 0) (color 0 0 0 0)
   )
@@
     (stroke (width 0) (type default))
   )
-  (wire (pts (xy 137.16 115.57) (xy 137.16 120.65))
+  (wire (pts (xy 29.21 74.93) (xy 36.83 74.93))
     (stroke (width 0) (type default))
   )
@@
     (stroke (width 0) (type default))
   )
+  (wire (pts (xy 127 118.11) (xy 137.16 118.11))
+    (stroke (width 0) (type default))
+  )
+  (wire (pts (xy 95.25 118.11) (xy 95.25 121.92))
+    (stroke (width 0) (type default))
+  )
   (wire (pts (xy 49.53 86.36) (xy 49.53 91.44))
     (stroke (width 0) (type default))
   )
-  (wire (pts (xy 120.65 77.47) (xy 120.65 87.63))
-    (stroke (width 0) (type default))
-  )
-  (wire (pts (xy 154.94 115.57) (xy 137.16 115.57))
+  (wire (pts (xy 120.65 77.47) (xy 120.65 81.28))
     (stroke (width 0) (type default))
   )
@@
     (stroke (width 0) (type default))
   )
-  (wire (pts (xy 137.16 115.57) (xy 137.16 100.33))
-    (stroke (width 0) (type default))
-  )
-  (wire (pts (xy 120.65 95.25) (xy 120.65 102.87))
+  (wire (pts (xy 137.16 100.33) (xy 137.16 118.11))
+    (stroke (width 0) (type default))
+  )
+  (wire (pts (xy 207.01 83.82) (xy 207.01 80.01))
+    (stroke (width 0) (type default))
+  )
+  (wire (pts (xy 120.65 88.9) (xy 120.65 90.17))
     (stroke (width 0) (type default))
   )
@@
     (stroke (width 0) (type default))
   )
-  (wire (pts (xy 120.65 110.49) (xy 120.65 113.03))
+  (wire (pts (xy 120.65 97.79) (xy 120.65 99.06))
     (stroke (width 0) (type default))
   )
@@
     (stroke (width 0) (type default))
   )
-  (wire (pts (xy 162.56 115.57) (xy 171.45 115.57))
+  (wire (pts (xy 119.38 118.11) (xy 110.49 118.11))
+    (stroke (width 0) (type default))
+  )
+  (wire (pts (xy 29.21 71.12) (xy 29.21 74.93))
     (stroke (width 0) (type default))
   )
@@
     (stroke (width 0) (type default))
   )
-  (wire (pts (xy 73.66 80.01) (xy 73.66 91.44))
+  (wire (pts (xy 73.66 80.01) (xy 73.66 88.9))
     (stroke (width 0) (type default))
   )
@@
     (stroke (width 0) (type default))
   )
+  (wire (pts (xy 137.16 118.11) (xy 137.16 120.65))
+    (stroke (width 0) (type default))
+  )
   (wire (pts (xy 185.42 80.01) (xy 185.42 86.36))
     (stroke (width 0) (type default))
   )
-  (wire (pts (xy 99.06 91.44) (xy 99.06 77.47))
+  (wire (pts (xy 99.06 88.9) (xy 99.06 77.47))
     (stroke (width 0) (type default))
   )
@@
     (stroke (width 0) (type default))
   )
+  (wire (pts (xy 95.25 118.11) (xy 102.87 118.11))
+    (stroke (width 0) (type default))
+  )
   (wire (pts (xy 115.57 77.47) (xy 120.65 77.47))
     (stroke (width 0) (type default))
   )
-  (wire (pts (xy 73.66 91.44) (xy 99.06 91.44))
+  (wire (pts (xy 73.66 88.9) (xy 99.06 88.9))
     (stroke (width 0) (type default))
   )
@@
     (stroke (width 0) (type default))
   )
-  (symbol (lib_id "power:GNDPWR") (at 120.65 113.03 0) (unit 1)
-    (in_bom yes) (on_board yes) (dnp no) (fields_autoplaced)
-    (property "Reference" "#PWR02" (at 120.65 118.11 0)
-      (effects (font (size 1.27 1.27)) hide)
-    )
-    (property "Value" "GNDPWR" (at 120.523 116.84 0)
-      (effects (font (size 1.27 1.27)))
-    )
-    (property "Footprint" "" (at 120.65 114.3 0)
-      (effects (font (size 1.27 1.27)) hide)
-    )
-    (property "Datasheet" "" (at 120.65 114.3 0)
+  (global_label "MID" (shape input) (at 95.25 118.11 180) (fields_autoplaced)
+    (effects (font (size 1.27 1.27)) (justify right))
+    (property "Intersheetrefs" "${INTERSHEET_REFS}" (at 88.9386 118.11 0)
+      (effects (font (size 1.27 1.27)) (justify right) hide)
+    )
+  )
+  (global_label "V_IN" (shape input) (at 29.21 74.93 180) (fields_autoplaced)
+    (effects (font (size 1.27 1.27)) (justify right))
+    (property "Intersheetrefs" "${INTERSHEET_REFS}" (at 22.2333 74.93 0)
+      (effects (font (size 1.27 1.27)) (justify right) hide)
+    )
+  )
+  (global_label "RNORM" (shape output) (at 207.01 80.01 0) (fields_autoplaced)
+    (effects (font (size 1.27 1.27)) (justify left))
+    (property "Intersheetrefs" "${INTERSHEET_REFS}" (at 216.6476 80.01 0)
+      (effects (font (size 1.27 1.27)) (justify left) hide)
+    )
+  )
+  (hierarchical_label "RNORM" (shape output) (at 207.01 83.82 0) (fields_autoplaced)
+    (effects (font (size 1.27 1.27)) (justify left))
+  )
+  (hierarchical_label "MID" (shape input) (at 95.25 121.92 180) (fields_autoplaced)
+    (effects (font (size 1.27 1.27)) (justify right))
+  )
+  (hierarchical_label "V_IN" (shape input) (at 29.21 71.12 180) (fields_autoplaced)
+    (effects (font (size 1.27 1.27)) (justify right))
+  )
+  (symbol (lib_id "power:GNDPWR") (at 120.65 99.06 0) (unit 1)
+    (in_bom yes) (on_board yes) (dnp no) (fields_autoplaced)
+    (property "Reference" "#PWR02" (at 120.65 104.14 0)
+      (effects (font (size 1.27 1.27)) hide)
+    )
+    (property "Value" "GNDPWR" (at 120.523 102.87 0)
+      (effects (font (size 1.27 1.27)))
+    )
+    (property "Footprint" "" (at 120.65 100.33 0)
+      (effects (font (size 1.27 1.27)) hide)
+    )
+    (property "Datasheet" "" (at 120.65 100.33 0)
       (effects (font (size 1.27 1.27)) hide)
     )
@@
     )
   )
-  (symbol (lib_id "Device:R") (at 175.26 115.57 90) (unit 1)
-    (in_bom yes) (on_board yes) (dnp no) (fields_autoplaced)
-    (property "Reference" "R8" (at 175.26 109.22 90)
-      (effects (font (size 1.27 1.27)))
-    )
-    (property "Value" "R" (at 175.26 111.76 90)
-      (effects (font (size 1.27 1.27)))
-    )
-    (property "Footprint" "" (at 175.26 117.348 90)
-      (effects (font (size 1.27 1.27)) hide)
-    )
-    (property "Datasheet" "~" (at 175.26 115.57 0)
+  (symbol (lib_id "Device:R") (at 106.68 118.11 270) (mirror x) (unit 1)
+    (in_bom yes) (on_board yes) (dnp no) (fields_autoplaced)
+    (property "Reference" "R8" (at 106.68 111.76 90)
+      (effects (font (size 1.27 1.27)))
+    )
+    (property "Value" "R" (at 106.68 114.3 90)
+      (effects (font (size 1.27 1.27)))
+    )
+    (property "Footprint" "" (at 106.68 119.888 90)
+      (effects (font (size 1.27 1.27)) hide)
+    )
+    (property "Datasheet" "~" (at 106.68 118.11 0)
       (effects (font (size 1.27 1.27)) hide)
     )
@@
     )
   )
-  (symbol (lib_id "Device:R") (at 158.75 115.57 90) (unit 1)
-    (in_bom yes) (on_board yes) (dnp no) (fields_autoplaced)
-    (property "Reference" "R7" (at 158.75 109.22 90)
-      (effects (font (size 1.27 1.27)))
-    )
-    (property "Value" "R" (at 158.75 111.76 90)
-      (effects (font (size 1.27 1.27)))
-    )
-    (property "Footprint" "" (at 158.75 117.348 90)
-      (effects (font (size 1.27 1.27)) hide)
-    )
-    (property "Datasheet" "~" (at 158.75 115.57 0)
+  (symbol (lib_id "Device:R") (at 123.19 118.11 270) (mirror x) (unit 1)
+    (in_bom yes) (on_board yes) (dnp no) (fields_autoplaced)
+    (property "Reference" "R7" (at 123.19 111.76 90)
+      (effects (font (size 1.27 1.27)))
+    )
+    (property "Value" "R" (at 123.19 114.3 90)
+      (effects (font (size 1.27 1.27)))
+    )
+    (property "Footprint" "" (at 123.19 119.888 90)
+      (effects (font (size 1.27 1.27)) hide)
+    )
+    (property "Datasheet" "~" (at 123.19 118.11 0)
       (effects (font (size 1.27 1.27)) hide)
     )
@@
     )
   )
-  (symbol (lib_id "Device:R") (at 120.65 91.44 180) (unit 1)
-    (in_bom yes) (on_board yes) (dnp no) (fields_autoplaced)
-    (property "Reference" "R5" (at 123.19 90.17 0)
-      (effects (font (size 1.27 1.27)) (justify right))
-    )
-    (property "Value" "R" (at 123.19 92.71 0)
-      (effects (font (size 1.27 1.27)) (justify right))
-    )
-    (property "Footprint" "" (at 122.428 91.44 90)
-      (effects (font (size 1.27 1.27)) hide)
-    )
-    (property "Datasheet" "~" (at 120.65 91.44 0)
+  (symbol (lib_id "Device:R") (at 120.65 85.09 180) (unit 1)
+    (in_bom yes) (on_board yes) (dnp no) (fields_autoplaced)
+    (property "Reference" "R5" (at 123.19 83.82 0)
+      (effects (font (size 1.27 1.27)) (justify right))
+    )
+    (property "Value" "R" (at 123.19 86.36 0)
+      (effects (font (size 1.27 1.27)) (justify right))
+    )
+    (property "Footprint" "" (at 122.428 85.09 90)
+      (effects (font (size 1.27 1.27)) hide)
+    )
+    (property "Datasheet" "~" (at 120.65 85.09 0)
       (effects (font (size 1.27 1.27)) hide)
     )
@@
     )
   )
-  (symbol (lib_id "Device:R") (at 120.65 106.68 180) (unit 1)
-    (in_bom yes) (on_board yes) (dnp no) (fields_autoplaced)
-    (property "Reference" "R6" (at 123.19 105.41 0)
-      (effects (font (size 1.27 1.27)) (justify right))
-    )
-    (property "Value" "R" (at 123.19 107.95 0)
-      (effects (font (size 1.27 1.27)) (justify right))
-    )
-    (property "Footprint" "" (at 122.428 106.68 90)
-      (effects (font (size 1.27 1.27)) hide)
-    )
-    (property "Datasheet" "~" (at 120.65 106.68 0)
-      (effects (font (size 1.27 1.27)) hide)
-    )
+  (symbol (lib_id "Device:R") (at 120.65 93.98 180) (unit 1)
+    (in_bom yes) (on_board yes) (dnp no) (fields_autoplaced)
+    (property "Reference" "R6" (at 123.19 92.71 0)
+      (effects (font (size 1.27 1.27)) (justify right))
+    )
+    (property "Value" "R" (at 123.19 95.25 0)
+      (effects (font (size 1.27 1.27)) (justify right))
+    )
+    (property "Footprint" "" (at 122.428 93.98 90)
+      (effects (font (size 1.27 1.27)) hide)
+    )
+    (property "Datasheet" "~" (at 120.65 93.98 0)
+      (effects (font (size 1.27 1.27)) hide)
+    )
