File: DNA/class_D/class_D_manual/class_D_manual.kicad_sch (KiCad schematic)
At the start: 0 parts

Commit message: [DNA]: class D, more of schematics added.
Other:
- added sheet Driver and half bridge (driver_half_bridge.kicad_sch)
- added sheet FPGA interface (fpga_interface.kicad_sch)
- added sheet Power (Power.kicad_sch)
- sheet Analog input ports: added MID, RNORM, V_IN; removed none
- sheet Feedback and compensation ports: added MID; removed none
- note added: "GND = 0 PGND = -10 LOGIC5 = -5 AUX5 = +5"
Changed lines of the file:
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@@
 (kicad_sch (version 20230121) (generator eeschema)
   (paper "A4")
-  (sheet (at 50.8 35.56) (size 20.32 8.89) (fields_autoplaced)
+  (wire (pts (xy 82.55 48.26) (xy 99.06 48.26))
+    (stroke (width 0) (type default))
+  )
+  (text "GND = 0\nPGND = -10\nLOGIC5 = -5\nAUX5 = +5" (at 217.17 40.64 0)
+    (effects (font (size 1.27 1.27)) (justify left bottom))
+  )
+  (sheet (at 99.06 39.37) (size 20.32 12.7) (fields_autoplaced)
     (stroke (width 0.1524) (type solid))
     (fill (color 0 0 0 0.0000))
-    (property "Sheetname" "Analog input" (at 50.8 34.8484 0)
+    (property "Sheetname" "Analog input" (at 99.06 38.6584 0)
       (effects (font (size 1.27 1.27)) (justify left bottom))
     )
-    (property "Sheetfile" "analog_input.kicad_sch" (at 50.8 45.0346 0)
+    (property "Sheetfile" "analog_input.kicad_sch" (at 99.06 52.6546 0)
       (effects (font (size 1.27 1.27)) (justify left top))
+    )
+    (pin "V_IN" input (at 99.06 43.18 180)
+      (effects (font (size 1.27 1.27)) (justify left))
+    )
+    (pin "RNORM" output (at 119.38 44.45 0)
+      (effects (font (size 1.27 1.27)) (justify right))
+    )
+    (pin "MID" input (at 99.06 48.26 180)
+      (effects (font (size 1.27 1.27)) (justify left))
     )
     (instances
@@
     )
   )
-  (sheet (at 53.34 68.58) (size 24.13 11.43) (fields_autoplaced)
+  (sheet (at 54.61 86.36) (size 24.13 11.43) (fields_autoplaced)
     (stroke (width 0.1524) (type solid))
     (fill (color 0 0 0 0.0000))
-    (property "Sheetname" "PWM and triangle generator" (at 53.34 67.8684 0)
+    (property "Sheetname" "PWM and triangle generator" (at 54.61 85.6484 0)
       (effects (font (size 1.27 1.27)) (justify left bottom))
     )
-    (property "Sheetfile" "pwm_gen.kicad_sch" (at 53.34 80.5946 0)
+    (property "Sheetfile" "pwm_gen.kicad_sch" (at 54.61 98.3746 0)
       (effects (font (size 1.27 1.27)) (justify left top))
     )
@@
     )
   )
-  (sheet (at 102.87 35.56) (size 26.67 12.7) (fields_autoplaced)
+  (sheet (at 53.34 114.3) (size 27.94 13.97) (fields_autoplaced)
     (stroke (width 0.1524) (type solid))
     (fill (color 0 0 0 0.0000))
-    (property "Sheetname" "Feedback and compensation" (at 102.87 34.8484 0)
+    (property "Sheetname" "FPGA interface" (at 53.34 113.5884 0)
       (effects (font (size 1.27 1.27)) (justify left bottom))
     )
-    (property "Sheetfile" "fb_and_comp.kicad_sch" (at 102.87 48.8446 0)
+    (property "Sheetfile" "fpga_interface.kicad_sch" (at 53.34 128.8546 0)
       (effects (font (size 1.27 1.27)) (justify left top))
+    )
+    (instances
+      (project "class_D_manual"
+        (path "/d93543c2-968a-4bbd-9580-bf9b3e26f4fe" (page "7"))
+      )
+    )
+  )
+  (sheet (at 41.91 39.37) (size 26.67 12.7) (fields_autoplaced)
+    (stroke (width 0.1524) (type solid))
+    (fill (color 0 0 0 0.0000))
+    (property "Sheetname" "Feedback and compensation" (at 41.91 38.6584 0)
+      (effects (font (size 1.27 1.27)) (justify left bottom))
+    )
+    (property "Sheetfile" "fb_and_comp.kicad_sch" (at 41.91 52.6546 0)
+      (effects (font (size 1.27 1.27)) (justify left top))
+    )
+    (pin "MID" input (at 41.91 44.45 180)
+      (effects (font (size 1.27 1.27)) (justify left))
     )
     (instances
@@
       )
     )
+  )
+  (sheet (at 101.6 86.36) (size 33.02 15.24) (fields_autoplaced)
+    (stroke (width 0.1524) (type solid))
+    (fill (color 0 0 0 0.0000))
+    (property "Sheetname" "Driver and half bridge" (at 101.6 85.6484 0)
+      (effects (font (size 1.27 1.27)) (justify left bottom))
+    )
+    (property "Sheetfile" "driver_half_bridge.kicad_sch" (at 101.6 102.1846 0)
+      (effects (font (size 1.27 1.27)) (justify left top))
+    )
+    (instances
+      (project "class_D_manual"
+        (path "/d93543c2-968a-4bbd-9580-bf9b3e26f4fe" (page "5"))
+      )
+    )
+  )
+  (sheet (at 153.67 87.63) (size 33.02 13.97) (fields_autoplaced)
+    (stroke (width 0.1524) (type solid))
+    (fill (color 0 0 0 0.0000))
+    (property "Sheetname" "Power" (at 153.67 86.9184 0)
+      (effects (font (size 1.27 1.27)) (justify left bottom))
+    )
+    (property "Sheetfile" "Power.kicad_sch" (at 153.67 102.1846 0)
+      (effects (font (size 1.27 1.27)) (justify left top))
+    )
+    (instances
+      (project "class_D_manual"
+        (path "/d93543c2-968a-4bbd-9580-bf9b3e26f4fe" (page "6"))
+      )
+    )
