File: DNA/class_D/class_D_manual/pwm_gen.kicad_sch (KiCad schematic)
At the start: 13 parts, among them U2 OPA810, U3 TLV3603

Commit message: [DNA]: class D, more of schematics added.
Parts:
- added R18: R, symbol Device:R
Connections:
- net LEAD: now reaches R13.1
- net CLK: now reaches C3.1
- net TRIANGLE: now reaches C4.2, C5.2, R12.2, U2.6, U3.2 (-)
- net RNORM: now reaches R14.1
- net LOGICS: now reaches R15.1
- net GNDPWR: now reaches R16.1
- net GNDPWR: now also R18.1
- net at R17.2, U3.6: now also R18.2
Changed lines of the file:
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@@
   (junction (at 106.68 40.64) (diameter 0) (color 0 0 0 0)
   )
+  (junction (at 118.11 73.66) (diameter 0) (color 0 0 0 0)
+  )
   (junction (at 76.2 40.64) (diameter 0) (color 0 0 0 0)
   )
@@
   (junction (at 137.16 129.54) (diameter 0) (color 0 0 0 0)
   )
+  (junction (at 180.34 101.6) (diameter 0) (color 0 0 0 0)
+  )
   (junction (at 76.2 71.12) (diameter 0) (color 0 0 0 0)
   )
@@
     (stroke (width 0) (type default))
   )
+  (wire (pts (xy 180.34 101.6) (xy 180.34 118.11))
+    (stroke (width 0) (type default))
+  )
   (wire (pts (xy 85.09 24.13) (xy 76.2 24.13))
     (stroke (width 0) (type default))
@@
     (stroke (width 0) (type default))
   )
+  (wire (pts (xy 106.68 115.57) (xy 114.3 115.57))
+    (stroke (width 0) (type default))
+  )
   (wire (pts (xy 85.09 54.61) (xy 76.2 54.61))
     (stroke (width 0) (type default))
@@
     (stroke (width 0) (type default))
   )
+  (wire (pts (xy 118.11 73.66) (xy 153.67 73.66))
+    (stroke (width 0) (type default))
+  )
   (wire (pts (xy 106.68 40.64) (xy 106.68 54.61))
     (stroke (width 0) (type default))
@@
     (stroke (width 0) (type default))
   )
+  (wire (pts (xy 118.11 64.77) (xy 118.11 73.66))
+    (stroke (width 0) (type default))
+  )
   (wire (pts (xy 53.34 71.12) (xy 62.23 71.12))
     (stroke (width 0) (type default))
   )
+  (wire (pts (xy 107.95 101.6) (xy 114.3 101.6))
+    (stroke (width 0) (type default))
+  )
   (wire (pts (xy 137.16 142.24) (xy 121.92 142.24))
     (stroke (width 0) (type default))
   )
-  (wire (pts (xy 106.68 73.66) (xy 153.67 73.66))
+  (wire (pts (xy 106.68 129.54) (xy 114.3 129.54))
+    (stroke (width 0) (type default))
+  )
+  (wire (pts (xy 110.49 144.78) (xy 110.49 142.24))
+    (stroke (width 0) (type default))
+  )
+  (wire (pts (xy 110.49 142.24) (xy 114.3 142.24))
+    (stroke (width 0) (type default))
+  )
+  (wire (pts (xy 106.68 73.66) (xy 118.11 73.66))
     (stroke (width 0) (type default))
   )
@@
     (stroke (width 0) (type default))
   )
+  (wire (pts (xy 24.13 71.12) (xy 27.94 71.12))
+    (stroke (width 0) (type default))
+  )
   (wire (pts (xy 76.2 40.64) (xy 76.2 54.61))
     (stroke (width 0) (type default))
@@
     (stroke (width 0) (type default))
   )
+  (wire (pts (xy 121.92 64.77) (xy 118.11 64.77))
+    (stroke (width 0) (type default))
+  )
   (wire (pts (xy 100.33 73.66) (xy 106.68 73.66))
     (stroke (width 0) (type default))
@@
     (stroke (width 0) (type default))
   )
+  (wire (pts (xy 180.34 125.73) (xy 180.34 132.08))
+    (stroke (width 0) (type default))
+  )
   (wire (pts (xy 76.2 54.61) (xy 76.2 71.12))
     (stroke (width 0) (type default))
   )
+  (global_label "TRIANGLE" (shape output) (at 121.92 64.77 0) (fields_autoplaced)
+    (effects (font (size 1.27 1.27)) (justify left))
+    (property "Intersheetrefs" "${INTERSHEET_REFS}" (at 133.6138 64.77 0)
+      (effects (font (size 1.27 1.27)) (justify left) hide)
+    )
+  )
+  (global_label "RNORM" (shape input) (at 106.68 115.57 180) (fields_autoplaced)
+    (effects (font (size 1.27 1.27)) (justify right))
+    (property "Intersheetrefs" "${INTERSHEET_REFS}" (at 97.0424 115.57 0)
+      (effects (font (size 1.27 1.27)) (justify right) hide)
+    )
+  )
+  (global_label "CLK" (shape input) (at 24.13 71.12 180) (fields_autoplaced)
+    (effects (font (size 1.27 1.27)) (justify right))
+    (property "Intersheetrefs" "${INTERSHEET_REFS}" (at 17.5767 71.12 0)
+      (effects (font (size 1.27 1.27)) (justify right) hide)
+    )
+  )
+  (global_label "LEAD" (shape input) (at 107.95 101.6 180) (fields_autoplaced)
+    (effects (font (size 1.27 1.27)) (justify right))
+    (property "Intersheetrefs" "${INTERSHEET_REFS}" (at 100.4291 101.6 0)
+      (effects (font (size 1.27 1.27)) (justify right) hide)
+    )
+  )
+  (global_label "LOGICS" (shape input) (at 106.68 129.54 180) (fields_autoplaced)
+    (effects (font (size 1.27 1.27)) (justify right))
+    (property "Intersheetrefs" "${INTERSHEET_REFS}" (at 96.9819 129.54 0)
+      (effects (font (size 1.27 1.27)) (justify right) hide)
+    )
+  )
   (symbol (lib_id "Device:R") (at 118.11 101.6 90) (unit 1)
     (in_bom yes) (on_board yes) (dnp no) (fields_autoplaced)
@@
         (path "/d93543c2-968a-4bbd-9580-bf9b3e26f4fe/25d8e2d5-2e70-4e34-a803-caf0c360ef09"
           (reference "R13") (unit 1)
+        )
+      )
+    )
+  )
+  (symbol (lib_id "Device:R") (at 180.34 121.92 180) (unit 1)
+    (in_bom yes) (on_board yes) (dnp no) (fields_autoplaced)
+    (property "Reference" "R18" (at 182.88 120.65 0)
+      (effects (font (size 1.27 1.27)) (justify right))
+    )
+    (property "Value" "R" (at 182.88 123.19 0)
+      (effects (font (size 1.27 1.27)) (justify right))
+    )
+    (property "Footprint" "" (at 182.118 121.92 90)
+      (effects (font (size 1.27 1.27)) hide)
+    )
+    (property "Datasheet" "~" (at 180.34 121.92 0)
+      (effects (font (size 1.27 1.27)) hide)
+    )
+    (pin "1")
+    (pin "2")
+    (instances
+      (project "class_D_manual"
+        (path "/d93543c2-968a-4bbd-9580-bf9b3e26f4fe/25d8e2d5-2e70-4e34-a803-caf0c360ef09"
+          (reference "R18") (unit 1)
         )
       )
@@
     )
   )
+  (symbol (lib_id "power:GNDPWR") (at 180.34 132.08 0) (unit 1)
+    (in_bom yes) (on_board yes) (dnp no) (fields_autoplaced)
+    (property "Reference" "#PWR06" (at 180.34 137.16 0)
+      (effects (font (size 1.27 1.27)) hide)
+    )
+    (property "Value" "GNDPWR" (at 180.213 135.89 0)
+      (effects (font (size 1.27 1.27)))
+    )
+    (property "Footprint" "" (at 180.34 133.35 0)
+      (effects (font (size 1.27 1.27)) hide)
+    )
+    (property "Datasheet" "" (at 180.34 133.35 0)
+      (effects (font (size 1.27 1.27)) hide)
+    )
+    (pin "1")
+    (instances
+      (project "class_D_manual"
+        (path "/d93543c2-968a-4bbd-9580-bf9b3e26f4fe/25d8e2d5-2e70-4e34-a803-caf0c360ef09"
+          (reference "#PWR06") (unit 1)
+        )
+      )
+    )
+  )
   (symbol (lib_id "Device:C") (at 88.9 54.61 90) (unit 1)
     (in_bom yes) (on_board yes) (dnp no) (fields_autoplaced)
@@
         )
       )
+    )
+  )
+  (symbol (lib_id "power:GNDPWR") (at 110.49 144.78 0) (unit 1)
+    (in_bom yes) (on_board yes) (dnp no) (fields_autoplaced)
+    (property "Reference" "#PWR05" (at 110.49 149.86 0)
+      (effects (font (size 1.27 1.27)) hide)
+    )
+    (property "Value" "GNDPWR" (at 110.363 148.59 0)
+      (effects (font (size 1.27 1.27)))
+    )
+    (property "Footprint" "" (at 110.49 146.05 0)
+      (effects (font (size 1.27 1.27)) hide)
+    )
+    (property "Datasheet" "" (at 110.49 146.05 0)
+      (effects (font (size 1.27 1.27)) hide)
+    )
+    (pin "1")
+    (instances
+      (project "class_D_manual"
+        (path "/d93543c2-968a-4bbd-9580-bf9b3e26f4fe/25d8e2d5-2e70-4e34-a803-caf0c360ef09"
+          (reference "#PWR05") (unit 1)
+        )
+      )
