File: DNA/class_B/class_B_manual/control.kicad_sch (KiCad schematic)
At the start: 16 parts, among them U1 OPA810IDBVR, U2 OPA810IDBVR

Commit message: [DNA]: all the schematics for Class B amplifier is ready.
TODO: 1. Add resistors', capacitors' values. 2. Add all footprints for resistors and connectors.
Other:
- moved on the sheet: C7, R7, R8, R9, U1

Commit message: [DNA]: class B: hierarchical labels added.
Changed lines of the file:
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@@
+    (stroke (width 0) (type default))
+  )
+  (wire (pts (xy 167.64 92.71) (xy 167.64 97.79))
     (stroke (width 0) (type default))
   )
@@
     (stroke (width 0) (type default))
   )
-  (wire (pts (xy 72.39 36.83) (xy 72.39 39.37))
+  (wire (pts (xy 72.39 33.02) (xy 72.39 39.37))
     (stroke (width 0) (type default))
   )
@@
     (stroke (width 0) (type default))
   )
+  (wire (pts (xy 45.72 58.42) (xy 46.99 58.42))
+    (stroke (width 0) (type default))
+  )
   (wire (pts (xy 72.39 46.99) (xy 72.39 52.07))
     (stroke (width 0) (type default))
@@
     (stroke (width 0) (type default))
   )
+  (wire (pts (xy 46.99 58.42) (xy 46.99 63.5))
+    (stroke (width 0) (type default))
+  )
+  (wire (pts (xy 44.45 69.85) (xy 44.45 73.66))
+    (stroke (width 0) (type default))
+  )
   (wire (pts (xy 186.69 81.28) (xy 198.12 81.28))
     (stroke (width 0) (type default))
@@
     (stroke (width 0) (type default))
   )
+  (wire (pts (xy 43.18 69.85) (xy 44.45 69.85))
+    (stroke (width 0) (type default))
+  )
   (wire (pts (xy 137.16 93.98) (xy 137.16 91.44))
     (stroke (width 0) (type default))
@@
     (stroke (width 0) (type default))
   )
+  (wire (pts (xy 71.12 33.02) (xy 72.39 33.02))
+    (stroke (width 0) (type default))
+  )
   (wire (pts (xy 130.81 91.44) (xy 137.16 91.44))
     (stroke (width 0) (type default))
@@
     (stroke (width 0) (type default))
   )
+  (wire (pts (xy 233.68 74.93) (xy 233.68 78.74))
+    (stroke (width 0) (type default))
+  )
   (wire (pts (xy 213.36 78.74) (xy 228.6 78.74))
     (stroke (width 0) (type default))
@@
     )
   )
+  (hierarchical_label "OUT_INT" (shape input) (at 45.72 58.42 180) (fields_autoplaced)
+    (effects (font (size 1.27 1.27)) (justify right))
+  )
+  (hierarchical_label "DRIVE" (shape input) (at 71.12 33.02 180) (fields_autoplaced)
+    (effects (font (size 1.27 1.27)) (justify right))
+  )
+  (hierarchical_label "LV_OUT" (shape output) (at 233.68 74.93 0) (fields_autoplaced)
+    (effects (font (size 1.27 1.27)) (justify left))
+  )
+  (hierarchical_label "V_REF" (shape input) (at 43.18 69.85 180) (fields_autoplaced)
+    (effects (font (size 1.27 1.27)) (justify right))
+  )
+  (hierarchical_label "VIN" (shape input) (at 167.64 92.71 180) (fields_autoplaced)
+    (effects (font (size 1.27 1.27)) (justify right))
+  )
   (symbol (lib_id "Device:R") (at 53.34 63.5 90) (unit 1)

Commit message: [DNA]: class B, resistor values etc added.
Parts:
- C5: value C -> 16.92n
- C6, C7: value C -> 4.7n
- C8: value C -> 1n
- R1: value R -> 27.7778
- R10: value R -> 470
- R2: value R -> 16.92k
- R3: value R -> 1k
- R4, R7: value R -> 100
- R5, R8: value R -> 330
- R6, R9: value R -> 1Meg
Other:
- note added: "!!! номиналы ненормальные"
Changed lines of the file:
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@@
     (stroke (width 0) (type default))
+  )
+  (text "!!! номиналы ненормальные\n\n" (at 36.83 95.25 0)
+    (effects (font (size 1.27 1.27)) (justify left bottom))
   )
   (global_label "+8V" (shape input) (at 95.25 68.58 0) (fields_autoplaced)
@@
       (effects (font (size 1.27 1.27)))
     )
-    (property "Value" "R" (at 53.34 59.69 90)
+    (property "Value" "16.92k" (at 53.34 59.69 90)
       (effects (font (size 1.27 1.27)))
     )
@@
       (effects (font (size 1.27 1.27)))
     )
-    (property "Value" "R" (at 217.17 93.98 90)
+    (property "Value" "330" (at 217.17 93.98 90)
       (effects (font (size 1.27 1.27)))
     )
@@
       (effects (font (size 1.27 1.27)) (justify left))
     )
-    (property "Value" "C" (at 76.2 44.45 0)
+    (property "Value" "1n" (at 76.2 44.45 0)
       (effects (font (size 1.27 1.27)) (justify left))
     )
@@
       (effects (font (size 1.27 1.27)) (justify right))
     )
-    (property "Value" "R" (at 139.7 99.06 0)
+    (property "Value" "1Meg" (at 139.7 99.06 0)
       (effects (font (size 1.27 1.27)) (justify right))
     )
@@
       (effects (font (size 1.27 1.27)) (justify left))
     )
-    (property "Value" "C" (at 125.73 99.06 0)
+    (property "Value" "4.7n" (at 125.73 99.06 0)
       (effects (font (size 1.27 1.27)) (justify left))
     )
@@
       (effects (font (size 1.27 1.27)) (justify left))
     )
-    (property "Value" "R" (at 74.93 102.87 0)
+    (property "Value" "27.7778" (at 74.93 102.87 0)
       (effects (font (size 1.27 1.27)) (justify left))
     )
@@
       (effects (font (size 1.27 1.27)) (justify left))
     )
-    (property "Value" "R" (at 74.93 57.15 0)
+    (property "Value" "470" (at 74.93 57.15 0)
       (effects (font (size 1.27 1.27)) (justify left))
     )
@@
       (effects (font (size 1.27 1.27)))
     )
-    (property "Value" "R" (at 53.34 69.85 90)
+    (property "Value" "1k" (at 53.34 69.85 90)
       (effects (font (size 1.27 1.27)))
     )
@@
       (effects (font (size 1.27 1.27)) (justify right))
     )
-    (property "Value" "R" (at 133.35 86.36 0)
+    (property "Value" "330" (at 133.35 86.36 0)
       (effects (font (size 1.27 1.27)) (justify right))
     )
@@
       (effects (font (size 1.27 1.27)))
     )
-    (property "Value" "R" (at 196.85 106.68 90)
+    (property "Value" "1Meg" (at 196.85 106.68 90)
       (effects (font (size 1.27 1.27)))
     )
@@
       (effects (font (size 1.27 1.27)))
     )
-    (property "Value" "R" (at 177.8 93.98 90)
+    (property "Value" "100" (at 177.8 93.98 90)
       (effects (font (size 1.27 1.27)))
     )
@@
       (effects (font (size 1.27 1.27)) (justify left))
     )
-    (property "Value" "C" (at 76.2 86.36 0)
+    (property "Value" "16.92n" (at 76.2 86.36 0)
       (effects (font (size 1.27 1.27)) (justify left))
     )
@@
       (effects (font (size 1.27 1.27)))
     )
-    (property "Value" "R" (at 120.65 72.39 90)
+    (property "Value" "100" (at 120.65 72.39 90)
       (effects (font (size 1.27 1.27)))
     )
@@
       (effects (font (size 1.27 1.27)))
     )
-    (property "Value" "C" (at 196.85 92.71 90)
-      (effects (font (size 1.27 1.27)))
-    )
+    (property "Value" "4.7n" (at 196.85 92.71 90)
+      (effects (font (size 1.27 1.27)))
+    )
