File: DNA/class_B/class_B_manual/diamond.kicad_sch (KiCad schematic)
At the start: 14 parts, among them Q4 FZTB53, Q5 FZTB53, Q6 FZT953, Q7 FZT953

Commit message: [DNA]: class B: hierarchical labels added.
Other:
- moved on the sheet: R21
Changed lines of the file:
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@@
   (junction (at 165.1 114.3) (diameter 0) (color 0 0 0 0)
   )
+  (junction (at 147.32 45.72) (diameter 0) (color 0 0 0 0)
+  )
   (junction (at 144.78 116.84) (diameter 0) (color 0 0 0 0)
   )
@@
   )
   (junction (at 198.12 101.6) (diameter 0) (color 0 0 0 0)
-  )
-  (junction (at 147.32 52.07) (diameter 0) (color 0 0 0 0)
   )
   (junction (at 173.99 55.88) (diameter 0) (color 0 0 0 0)
@@
     (stroke (width 0) (type default))
   )
-  (wire (pts (xy 147.32 52.07) (xy 147.32 55.88))
-    (stroke (width 0) (type default))
-  )
   (wire (pts (xy 144.78 116.84) (xy 144.78 119.38))
     (stroke (width 0) (type default))
@@
     (stroke (width 0) (type default))
   )
+  (wire (pts (xy 83.82 77.47) (xy 83.82 82.55))
+    (stroke (width 0) (type default))
+  )
   (wire (pts (xy 177.8 91.44) (xy 177.8 93.98))
     (stroke (width 0) (type default))
@@
     (stroke (width 0) (type default))
   )
-  (wire (pts (xy 124.46 45.72) (xy 143.51 45.72))
+  (wire (pts (xy 124.46 45.72) (xy 147.32 45.72))
     (stroke (width 0) (type default))
   )
@@
     (stroke (width 0) (type default))
   )
-  (wire (pts (xy 143.51 52.07) (xy 147.32 52.07))
-    (stroke (width 0) (type default))
-  )
   (wire (pts (xy 124.46 109.22) (xy 137.16 109.22))
     (stroke (width 0) (type default))
@@
     (stroke (width 0) (type default))
   )
+  (wire (pts (xy 147.32 45.72) (xy 147.32 55.88))
+    (stroke (width 0) (type default))
+  )
   (wire (pts (xy 147.32 66.04) (xy 147.32 69.85))
     (stroke (width 0) (type default))
@@
     (stroke (width 0) (type default))
   )
-  (wire (pts (xy 147.32 39.37) (xy 147.32 43.18))
+  (wire (pts (xy 147.32 30.48) (xy 147.32 34.29))
     (stroke (width 0) (type default))
   )
@@
     (stroke (width 0) (type default))
   )
+  (wire (pts (xy 210.82 78.74) (xy 210.82 83.82))
+    (stroke (width 0) (type default))
+  )
   (wire (pts (xy 165.1 114.3) (xy 165.1 91.44))
     (stroke (width 0) (type default))
@@
     (stroke (width 0) (type default))
   )
-  (wire (pts (xy 143.51 45.72) (xy 143.51 52.07))
-    (stroke (width 0) (type default))
-  )
-  (wire (pts (xy 147.32 50.8) (xy 147.32 52.07))
+  (wire (pts (xy 147.32 41.91) (xy 147.32 45.72))
     (stroke (width 0) (type default))
   )
@@
     )
   )
-  (global_label "+50V" (shape bidirectional) (at 147.32 39.37 0) (fields_autoplaced)
-    (effects (font (size 1.27 1.27)) (justify left))
-    (property "Intersheetrefs" "${INTERSHEET_REFS}" (at 156.4965 39.37 0)
+  (global_label "+50V" (shape bidirectional) (at 147.32 30.48 0) (fields_autoplaced)
+    (effects (font (size 1.27 1.27)) (justify left))
+    (property "Intersheetrefs" "${INTERSHEET_REFS}" (at 156.4965 30.48 0)
       (effects (font (size 1.27 1.27)) (justify left) hide)
     )
@@
       (effects (font (size 1.27 1.27)) (justify left) hide)
     )
+  )
+  (hierarchical_label "VAS_OUT" (shape input) (at 83.82 77.47 180) (fields_autoplaced)
+    (effects (font (size 1.27 1.27)) (justify right))
+  )
+  (hierarchical_label "DRIVE" (shape output) (at 210.82 78.74 0) (fields_autoplaced)
+    (effects (font (size 1.27 1.27)) (justify left))
   )
   (symbol (lib_id "Diode:BAV99") (at 129.54 124.46 270) (unit 1)
@@
     )
   )
-  (symbol (lib_id "Device:R") (at 147.32 46.99 0) (unit 1)
-    (in_bom yes) (on_board yes) (dnp no) (fields_autoplaced)
-    (property "Reference" "R21" (at 149.86 45.72 0)
-      (effects (font (size 1.27 1.27)) (justify left))
-    )
-    (property "Value" "R" (at 149.86 48.26 0)
-      (effects (font (size 1.27 1.27)) (justify left))
-    )
-    (property "Footprint" "" (at 145.542 46.99 90)
-      (effects (font (size 1.27 1.27)) hide)
-    )
-    (property "Datasheet" "~" (at 147.32 46.99 0)
-      (effects (font (size 1.27 1.27)) hide)
-    )
+  (symbol (lib_id "Device:R") (at 147.32 38.1 0) (unit 1)
+    (in_bom yes) (on_board yes) (dnp no) (fields_autoplaced)
+    (property "Reference" "R21" (at 149.86 36.83 0)
+      (effects (font (size 1.27 1.27)) (justify left))
+    )
+    (property "Value" "R" (at 149.86 39.37 0)
+      (effects (font (size 1.27 1.27)) (justify left))
+    )
+    (property "Footprint" "" (at 145.542 38.1 90)
+      (effects (font (size 1.27 1.27)) hide)
+    )
+    (property "Datasheet" "~" (at 147.32 38.1 0)
+      (effects (font (size 1.27 1.27)) hide)
+    )

Commit message: [DNA]: class B, resistor values etc added.
Parts:
- R17, R18: value R -> 2.2
- R19, R21: value R -> 2.2k
- R20, R22: value R -> 10
Changed lines of the file:
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@@
       (effects (font (size 1.27 1.27)) (justify left))
     )
-    (property "Value" "R" (at 147.32 124.46 0)
+    (property "Value" "2.2k" (at 147.32 124.46 0)
       (effects (font (size 1.27 1.27)) (justify left))
     )
@@
       (effects (font (size 1.27 1.27)) (justify left))
     )
-    (property "Value" "R" (at 200.66 72.39 0)
+    (property "Value" "2.2" (at 200.66 72.39 0)
       (effects (font (size 1.27 1.27)) (justify left))
     )
@@
       (effects (font (size 1.27 1.27)))
     )
-    (property "Value" "R" (at 114.3 105.41 90)
+    (property "Value" "10" (at 114.3 105.41 90)
       (effects (font (size 1.27 1.27)))
     )
@@
       (effects (font (size 1.27 1.27)) (justify left))
     )
-    (property "Value" "R" (at 149.86 39.37 0)
+    (property "Value" "2.2k" (at 149.86 39.37 0)
       (effects (font (size 1.27 1.27)) (justify left))
     )
@@
       (effects (font (size 1.27 1.27)))
     )
-    (property "Value" "R" (at 107.95 57.15 90)
+    (property "Value" "10" (at 107.95 57.15 90)
       (effects (font (size 1.27 1.27)))
     )
@@
       (effects (font (size 1.27 1.27)) (justify left))
     )
-    (property "Value" "R" (at 200.66 97.79 0)
-      (effects (font (size 1.27 1.27)) (justify left))
-    )
+    (property "Value" "2.2" (at 200.66 97.79 0)
+      (effects (font (size 1.27 1.27)) (justify left))
+    )
