File: DNA/class_B/class_B_manual/power.kicad_sch (KiCad schematic)
At the start: 21 parts, among them Q10 2N5551, Q11 2N5401, Q8 MJL3281A, Q9 MJL1302A

Commit message: [DNA]: class B: hierarchical labels added.
Changed lines of the file:
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@@
   (junction (at 166.37 96.52) (diameter 0) (color 0 0 0 0)
+  )
+  (junction (at 182.88 90.17) (diameter 0) (color 0 0 0 0)
   )
   (junction (at 120.65 123.19) (diameter 0) (color 0 0 0 0)
@@
     (stroke (width 0) (type default))
   )
+  (wire (pts (xy 184.15 85.09) (xy 182.88 85.09))
+    (stroke (width 0) (type default))
+  )
   (wire (pts (xy 80.01 128.27) (xy 88.9 128.27))
     (stroke (width 0) (type default))
@@
     (stroke (width 0) (type default))
   )
+  (wire (pts (xy 182.88 85.09) (xy 182.88 90.17))
+    (stroke (width 0) (type default))
+  )
   (wire (pts (xy 104.14 46.99) (xy 104.14 64.77))
     (stroke (width 0) (type default))
@@
     (stroke (width 0) (type default))
   )
+  (wire (pts (xy 232.41 91.44) (xy 232.41 96.52))
+    (stroke (width 0) (type default))
+  )
   (wire (pts (xy 182.88 90.17) (xy 182.88 96.52))
     (stroke (width 0) (type default))
@@
   )
   (wire (pts (xy 80.01 96.52) (xy 80.01 128.27))
+    (stroke (width 0) (type default))
+  )
+  (wire (pts (xy 67.31 92.71) (xy 67.31 96.52))
     (stroke (width 0) (type default))
   )
@@
     )
   )
+  (hierarchical_label "OUT_INT" (shape output) (at 184.15 85.09 0) (fields_autoplaced)
+    (effects (font (size 1.27 1.27)) (justify left))
+  )
+  (hierarchical_label "COM" (shape output) (at 232.41 91.44 0) (fields_autoplaced)
+    (effects (font (size 1.27 1.27)) (justify left))
+  )
+  (hierarchical_label "DRIVE" (shape input) (at 67.31 92.71 180) (fields_autoplaced)
+    (effects (font (size 1.27 1.27)) (justify right))
+  )
   (symbol (lib_id "Device:R") (at 137.16 123.19 90) (unit 1)

Commit message: [DNA]: class B, resistor values etc added.
Parts:
- L1: value L -> 100n / DCR 20m
- R23, R25: value R -> 2.2
- R24, R26: value R -> 10
- R27, R28: value R -> 4.7
- R29: value R -> 22
- R30, R31: value R -> 0.22
- R32: value R -> 0.47
Changed lines of the file:
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@@
       (effects (font (size 1.27 1.27)))
     )
-    (property "Value" "R" (at 137.16 119.38 90)
+    (property "Value" "2.2" (at 137.16 119.38 90)
       (effects (font (size 1.27 1.27)))
     )
@@
       (effects (font (size 1.27 1.27)))
     )
-    (property "Value" "R" (at 92.71 124.46 90)
+    (property "Value" "4.7" (at 92.71 124.46 90)
       (effects (font (size 1.27 1.27)))
     )
@@
       (effects (font (size 1.27 1.27)))
     )
-    (property "Value" "R" (at 92.71 92.71 90)
+    (property "Value" "22" (at 92.71 92.71 90)
       (effects (font (size 1.27 1.27)))
     )
@@
       (effects (font (size 1.27 1.27)))
     )
-    (property "Value" "R" (at 90.17 60.96 90)
+    (property "Value" "4.7" (at 90.17 60.96 90)
       (effects (font (size 1.27 1.27)))
     )
@@
       (effects (font (size 1.27 1.27)))
     )
-    (property "Value" "L" (at 209.55 93.98 90)
+    (property "Value" "100n / DCR 20m" (at 209.55 93.98 90)
       (effects (font (size 1.27 1.27)))
     )
@@
       (effects (font (size 1.27 1.27)) (justify right))
     )
-    (property "Value" "R" (at 123.19 82.55 0)
+    (property "Value" "0.22" (at 123.19 82.55 0)
       (effects (font (size 1.27 1.27)) (justify right))
     )
@@
       (effects (font (size 1.27 1.27)))
     )
-    (property "Value" "R" (at 154.94 74.93 90)
+    (property "Value" "10" (at 154.94 74.93 90)
       (effects (font (size 1.27 1.27)))
     )
@@
       (effects (font (size 1.27 1.27)) (justify right))
     )
-    (property "Value" "R" (at 123.19 110.49 0)
+    (property "Value" "0.22" (at 123.19 110.49 0)
       (effects (font (size 1.27 1.27)) (justify right))
     )
@@
       (effects (font (size 1.27 1.27)))
     )
-    (property "Value" "R" (at 157.48 107.95 90)
+    (property "Value" "10" (at 157.48 107.95 90)
       (effects (font (size 1.27 1.27)))
     )
@@
       (effects (font (size 1.27 1.27)))
     )
-    (property "Value" "R" (at 138.43 66.04 90)
+    (property "Value" "2.2" (at 138.43 66.04 90)
       (effects (font (size 1.27 1.27)))
     )
@@
       (effects (font (size 1.27 1.27)))
     )
-    (property "Value" "R" (at 209.55 104.14 90)
-      (effects (font (size 1.27 1.27)))
-    )
+    (property "Value" "0.47" (at 209.55 104.14 90)
+      (effects (font (size 1.27 1.27)))
+    )
